File: TinyLilFucker.kicad_pcb (KiCad board)
At the start: 2 copper layers, 28.5 x 17.5 mm, 11 parts, among them J1 USB_A, J2 Conn_02x05_Top_Bottom, U1 STM32C071F8Px, U2 AP2112K-3.3TRG1

Commit message: Rename text from 'TINYLILFUCKER' to 'TINYLILFELLA'
Other:
- board text added: "TINYLILFELLA MADE BY YURI YERMOL"
- board text removed: "TINYLILFUCKER MADE BY YURI YERMOL"
Changed lines of the file:
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@@
 		(layer "Edge.Cuts")
 	)
-	(gr_text "TINYLILFUCKER\nMADE BY YURI YERMOL"
+	(gr_text "TINYLILFELLA\nMADE BY YURI YERMOL"
 		(at 44.5 27.5 0)
 		(layer "F.SilkS")

Commit message: Add files via upload
Parts:
- added ?: , , F.Cu at (41.0, 12.0)
- added ?: , , F.Cu at (66.5, 12.0)
- added ?: , , F.Cu at (66.5, 26.5)
Changed lines of the file:
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@@
 		)
+	)
+	(footprint ""
+		(layer "F.Cu")
+		(at 41 12)
+		(property "Reference" ""
+			(at 0 0 0)
+			(layer "F.SilkS")
+			(effects
+				(font
+					(size 1.27 1.27)
+				)
+			)
+		)
+		(property "Value" ""
+			(at 0 0 0)
+			(layer "F.Fab")
+			(effects
+				(font
+					(size 1.27 1.27)
+				)
+			)
+		)
+		(property "Datasheet" ""
+			(at 0 0 0)
+			(layer "F.Fab")
+			(hide yes)
+			(effects
+				(font
+					(size 1.27 1.27)
+				)
+			)
+		)
+		(property "Description" ""
+			(at 0 0 0)
+			(layer "F.Fab")
+			(hide yes)
+			(effects
+				(font
+					(size 1.27 1.27)
+				)
+			)
+		)
+		(duplicate_pad_numbers_are_jumpers no)
+		(pad "" np_thru_hole circle
+			(at 0 0)
+			(size 2.1 2.1)
+			(drill 1.8)
+			(layers "*.Cu" "*.Mask")
+		)
+		(embedded_fonts no)
 	)
 	(footprint "Package_SO:TSSOP-20_4.4x6.5mm_P0.65mm"
@@
 		)
 	)
+	(footprint ""
+		(layer "F.Cu")
+		(at 66.5 12)
+		(property "Reference" ""
+			(at 0 0 0)
+			(layer "F.SilkS")
+			(effects
+				(font
+					(size 1.27 1.27)
+				)
+			)
+		)
+		(property "Value" ""
+			(at 0 0 0)
+			(layer "F.Fab")
+			(effects
+				(font
+					(size 1.27 1.27)
+				)
+			)
+		)
+		(property "Datasheet" ""
+			(at 0 0 0)
+			(layer "F.Fab")
+			(hide yes)
+			(effects
+				(font
+					(size 1.27 1.27)
+				)
+			)
+		)
+		(property "Description" ""
+			(at 0 0 0)
+			(layer "F.Fab")
+			(hide yes)
+			(effects
+				(font
+					(size 1.27 1.27)
+				)
+			)
+		)
+		(duplicate_pad_numbers_are_jumpers no)
+		(pad "" np_thru_hole circle
+			(at 0 0)
+			(size 2.1 2.1)
+			(drill 1.8)
+			(layers "*.Cu" "*.Mask")
+		)
+		(embedded_fonts no)
+	)
 	(footprint "LED_SMD:LED_Cree-PLCC4_2x2mm_CW"
 		(layer "F.Cu")
@@
 		)
 	)
+	(footprint ""
+		(layer "F.Cu")
+		(at 66.5 26.5)
+		(property "Reference" ""
+			(at 0 0 0)
+			(layer "F.SilkS")
+			(effects
+				(font
+					(size 1.27 1.27)
+				)
+			)
+		)
+		(property "Value" ""
+			(at 0 0 0)
+			(layer "F.Fab")
+			(effects
+				(font
+					(size 1.27 1.27)
+				)
+			)
+		)
+		(property "Datasheet" ""
+			(at 0 0 0)
+			(layer "F.Fab")
+			(hide yes)
+			(effects
+				(font
+					(size 1.27 1.27)
+				)
+			)
+		)
+		(property "Description" ""
+			(at 0 0 0)
+			(layer "F.Fab")
+			(hide yes)
+			(effects
+				(font
+					(size 1.27 1.27)
+				)
+			)
+		)
+		(duplicate_pad_numbers_are_jumpers no)
+		(pad "" np_thru_hole circle
+			(at 0 0)
+			(size 2.1 2.1)
+			(drill 1.8)
+			(layers "*.Cu" "*.Mask")
+		)
+		(embedded_fonts no)
+	)
 	(footprint "Connector_USB:USB_A_Connfly_DS1098_Horizontal"
