File: files/TinyLilFucker.kicad_sch (KiCad schematic)
At the start: 11 parts, among them J1 USB_A, J2 Conn_02x05_Top_Bottom, SW1 SW_Push, U1 STM32C071F8Px, U2 AP2112K-3.3TRG1

Commit message: Add files via upload
Parts:
- added LED2: LED_SMD_1W_3W, LED_SMD:LED_01005_0402Metric, symbol PCM_LED_AKL:LED_SMD_1W_3W
- added R1: 1k, Resistor_SMD:R_01005_0402Metric, symbol PCM_SL_Resistors:1k
Connections:
- net at J1.1 (VBUS), J2.4 (Pin_4), U2.1 (IN)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: now also R1.1
- net at C2.2, J1.4 (GND), J1.SH (Shield)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: now also LED2.1 (K)
- new net: LED2.2 (A), R1.2
Changed lines of the file:
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@@
+	)
+	(junction
+		(at 46.99 40.64)
+		(diameter 0)
+		(color 0 0 0 0)
 	)
 	(junction
@@
 	)
 	(junction
+		(at 30.48 21.59)
+		(diameter 0)
+		(color 0 0 0 0)
+	)
+	(junction
 		(at 52.07 68.58)
 		(diameter 0)
@@
 	(wire
 		(pts
+			(xy 31.75 40.64) (xy 31.75 21.59)
+		)
+		(stroke
+			(width 0)
+			(type default)
+		)
+	)
+	(wire
+		(pts
 			(xy 59.69 72.39) (xy 59.69 43.18)
 		)
@@
 	(wire
 		(pts
-			(xy 46.99 34.29) (xy 46.99 68.58)
+			(xy 46.99 34.29) (xy 46.99 40.64)
 		)
 		(stroke
@@
 	(wire
 		(pts
+			(xy 31.75 21.59) (xy 30.48 21.59)
+		)
+		(stroke
+			(width 0)
+			(type default)
+		)
+	)
+	(wire
+		(pts
 			(xy 52.07 68.58) (xy 80.01 68.58)
 		)
@@
 		(pts
 			(xy 149.86 40.64) (xy 154.94 40.64)
+		)
+		(stroke
+			(width 0)
+			(type default)
+		)
+	)
+	(wire
+		(pts
+			(xy 46.99 40.64) (xy 46.99 68.58)
 		)
 		(stroke
@@
 	)
 	(symbol
+		(lib_id "PCM_LED_AKL:LED_SMD_1W_3W")
+		(at 43.18 40.64 0)
+		(unit 1)
+		(body_style 1)
+		(exclude_from_sim no)
+		(in_bom yes)
+		(on_board yes)
+		(in_pos_files yes)
+		(dnp no)
+		(fields_autoplaced yes)
+		(property "Reference" "LED2"
+			(at 43.18 31.75 0)
+			(show_name no)
+			(do_not_autoplace no)
+			(effects
+				(font
+					(size 1.27 1.27)
+				)
+			)
+		)
+		(property "Value" "LED_SMD_1W_3W"
+			(at 43.18 34.29 0)
+			(show_name no)
+			(do_not_autoplace no)
+			(effects
+				(font
+					(size 1.27 1.27)
+				)
+			)
+		)
+		(property "Footprint" "LED_SMD:LED_01005_0402Metric"
+			(at 43.18 40.64 0)
+			(hide yes)
+			(show_name no)
+			(do_not_autoplace no)
+			(effects
+				(font
+					(size 1.27 1.27)
+				)
+			)
+		)
+		(property "Datasheet" ""
+			(at 43.18 40.64 0)
+			(hide yes)
+			(show_name no)
+			(do_not_autoplace no)
+			(effects
+				(font
+					(size 1.27 1.27)
+				)
+			)
+		)
+		(property "Description" "SMD Power LED, Generic, Alternate KiCad Library"
+			(at 43.18 40.64 0)
+			(hide yes)
+			(show_name no)
+			(do_not_autoplace no)
+			(effects
+				(font
+					(size 1.27 1.27)
+				)
+			)
+		)
+		(pin "2"
+		)
+		(pin "1"
+		)
+		(instances
+			(project "TinyLilFucker"
+				(path "/03c9d907-95d7-4615-9b71-a13bb7438c3c"
+					(reference "LED2")
+					(unit 1)
+				)
+			)
+		)
+	)
+	(symbol
 		(lib_id "Connector:USB_A")
 		(at 22.86 26.67 0)
@@
 					(unit 1)
 				)
+			)
+		)
+	)
+	(symbol
+		(lib_id "PCM_SL_Resistors:1k")
+		(at 35.56 40.64 0)
+		(unit 1)
+		(body_style 1)
+		(exclude_from_sim no)
+		(in_bom yes)
+		(on_board yes)
+		(in_pos_files yes)
+		(dnp no)
+		(fields_autoplaced yes)
+		(property "Reference" "R1"
+			(at 35.56 34.29 0)
+			(show_name no)
+			(do_not_autoplace no)
+			(effects
+				(font
+					(size 1.27 1.27)
+				)
+			)
+		)
+		(property "Value" "1k"
+			(at 35.56 36.83 0)
+			(show_name no)
+			(do_not_autoplace no)
+			(effects
+				(font
+					(size 1.27 1.27)
+				)
+			)
+		)
+		(property "Footprint" "Resistor_SMD:R_01005_0402Metric"
+			(at 36.449 44.958 0)
+			(hide yes)
+			(show_name no)
+			(do_not_autoplace no)
+			(effects
+				(font
+					(size 1.27 1.27)
+				)
+			)
+		)
+		(property "Datasheet" ""
+			(at 36.068 40.64 0)
+			(hide yes)
+			(show_name no)
+			(do_not_autoplace no)
+			(effects
+				(font
+					(size 1.27 1.27)
+				)
+			)
+		)
+		(property "Description" "1kΩ, 1/4W Resistor"
+			(at 35.56 40.64 0)
+			(hide yes)
+			(show_name no)
+			(do_not_autoplace no)
+			(effects
+				(font
+					(size 1.27 1.27)
+				)
+			)
+		)
+		(pin "1"
+		)
+		(pin "2"
+		)
+		(instances
+			(project "TinyLilFucker"
+				(path "/03c9d907-95d7-4615-9b71-a13bb7438c3c"
+					(reference "R1")
+					(unit 1)
+				)
