File: files/TinyLilFucker.kicad_pcb (KiCad board)
At the start: 2 copper layers, 28.5 x 17.5 mm, 14 parts, among them J1 USB_A, J2 Conn_02x05_Top_Bottom, U1 STM32C071F8Px, U2 AP2112K-3.3TRG1

Commit message: Add files via upload
Parts:
- added LED2: LED_SMD_1W_3W, LED_SMD:LED_01005_0402Metric, B.Cu at (45.8, 27.0)
- added R1: 1k, Resistor_SMD:R_01005_0402Metric, B.Cu at (47.8, 27.0)
- C1: value (none) -> 10uF_16V
- C2: value (none) -> 100uF_10V
- SW1: value (none) -> SW_Push
Routing:
- net Net-(J1-VBUS): track 23.0 -> 42.6 mm, vias 0 -> 2
- net Net-(J1-GND): track 73.1 -> 77.2 mm
- net Net-(LED2-A): track 0.00 -> 2.51 mm
Other:
- board size 28.5 x 17.5 mm -> 28.5 x 19.5 mm
- board text added: "PWR"

Commit message: Add files via upload
Parts:
- moved ? 26.0 mm to (40.8, 29.8)
- moved ? 3.26 mm to (69.8, 11.8)
- moved ? 0.35 mm to (40.8, 11.8)
Other:
- board size 28.5 x 19.5 mm -> 31.5 x 20.5 mm
- board text added: "GITHUB @PURPLETUE A PART OF HACK CLUB STARDANCE"
- board text removed: "STM32"

Commit message: Add files via upload
Other:
- board text added: "STM32C071"
